Commit message: enable debug

File: rexrov2_description/urdf/rexrov2.gazebo.xacro (robot description, xacro)
@@ -19,6 +19,8 @@
     -->
     <xacro:property name="cob" value="0.0 0.0 0.3"/>
+    <!--<xacro:property name="cob" value="0.0 0.0 0.0"/>-->
     <!-- Volume, see p.31 in Berg2012 -->
     <xacro:property name="volume" value="1.83826"/>
+    <!--<xacro:property name="volume" value="1.8121303501945525"/>-->
     <xacro:macro name="rexrov2_hydro_model" params="namespace">
         <link name="${namespace}/base_link">
