Commit message: various confgurations of rexrov2 for different experiments

File: rexrov2_description/urdf/rexrov2_diag_pos.gazebo.xacro (robot description, xacro)
@@ -21,5 +21,5 @@
     <!--<xacro:property name="cob" value="0.0 0.0 0.0"/>-->
     <!-- Volume, see p.31 in Berg2012 -->
-    <xacro:property name="volume" value="1.8121303501945525"/>
+    <xacro:property name="volume" value="1.83826"/>
     <xacro:macro name="rexrov2_hydro_model" params="namespace">
         <link name="${namespace}/base_link">
